File: RaceTracker.kicad_prj/GPS.kicad_sch (KiCad schematic)
At the start: 23 parts, among them U103 ZED-F9P RTK GNSS

Commit message: Footprints für GPS+Sensors_Storage: 132/132 Bauteile jetzt komplett
GPS-Blatt: SMA_EDGE, ML414H_COIN_CELL und ZED_F9P_LGA102 (bereits
vorhandene Custom-Footprints) verlinkt, Pad-Namen gegen Schaltplan-Pins
verifiziert. Restliche Passiva auf Standardbibliothek gemappt.

Sensors_Storage-Blatt: U7 (MPU-6050) auf KiCads eigene
Sensor_Motion:InvenSense_QFN-24_4x4mm_P0.5mm (exakt für diesen Chip
vorgesehen, nicht generisch geraten). J10 (MicroSD) auf
Connector_Card:microSD_HC_Molex_104031-0811 (Industriestandard-Teil).
J11 (e-Paper) auf 2,54mm-8-Pin-Stiftleiste, passend zum "steckbar"-Debug-
Anschluss von Waveshare-e-Paper-Modulen.

Damit haben alle 132 Bauteile im Projekt ein Footprint (vorher 1/132).
ERC weiterhin 0 Fehler/0 Warnungen, inklusive Footprint-Bibliotheksprüfung.

Co-Authored-By: Claude Sonnet 5 <noreply@anthropic.com>
Parts:
- B101: footprint (none) -> RaceTracker:ML414H_COIN_CELL
- C101, C103, C104, C105, C107: footprint (none) -> Capacitor_SMD:C_0402_1005Metric
- D101, D103, D104: footprint (none) -> RaceTracker:LED_0603_AK
- D102: footprint (none) -> RaceTracker:SODFL3517X110N
- E101: footprint (none) -> RaceTracker:SMA_EDGE
- FB101: footprint (none) -> Inductor_SMD:L_0402_1005Metric
- R105, R107, R108, R111, R112, R113, R114, R121, R124, R125: footprint (none) -> Resistor_SMD:R_0402_1005Metric
- U103: footprint (none) -> RaceTracker:ZED_F9P_LGA102
Changed lines of the file:
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@@
 			)
 		)
-		(property "Footprint" ""
+		(property "Footprint" "Capacitor_SMD:C_0402_1005Metric"
 			(at 109.22 54.61 0)
 			(hide yes)
@@
 			)
 		)
-		(property "Footprint" ""
+		(property "Footprint" "RaceTracker:LED_0603_AK"
 			(at 165.1 107.95 0)
 			(hide yes)
@@
 			)
 		)
-		(property "Footprint" ""
+		(property "Footprint" "Resistor_SMD:R_0402_1005Metric"
 			(at 251.46 54.61 0)
 			(hide yes)
@@
 			)
 		)
-		(property "Footprint" ""
+		(property "Footprint" "Resistor_SMD:R_0402_1005Metric"
 			(at 124.46 107.95 0)
 			(hide yes)
@@
 			)
 		)
-		(property "Footprint" ""
+		(property "Footprint" "RaceTracker:SMA_EDGE"
 			(at 190.5 54.61 0)
 			(hide yes)
@@
 			)
 		)
-		(property "Footprint" ""
+		(property "Footprint" "Inductor_SMD:L_0402_1005Metric"
 			(at 149.86 54.61 0)
 			(hide yes)
@@
 			)
 		)
-		(property "Footprint" ""
+		(property "Footprint" "Resistor_SMD:R_0402_1005Metric"
 			(at 144.78 107.95 0)
 			(hide yes)
@@
 			)
 		)
-		(property "Footprint" ""
+		(property "Footprint" "Capacitor_SMD:C_0402_1005Metric"
 			(at 88.9 54.61 0)
 			(hide yes)
@@
 			)
 		)
-		(property "Footprint" ""
+		(property "Footprint" "Capacitor_SMD:C_0402_1005Metric"
 			(at 231.14 54.61 0)
 			(hide yes)
@@
 			)
 		)
-		(property "Footprint" ""
+		(property "Footprint" "RaceTracker:ML414H_COIN_CELL"
 			(at 210.82 54.61 0)
 			(hide yes)
@@
 			)
 		)
-		(property "Footprint" ""
+		(property "Footprint" "RaceTracker:LED_0603_AK"
 			(at 226.06 107.95 0)
 			(hide yes)
@@
 			)
 		)
-		(property "Footprint" ""
+		(property "Footprint" "Resistor_SMD:R_0402_1005Metric"
 			(at 205.74 107.95 0)
 			(hide yes)
@@
 			)
 		)
-		(property "Footprint" ""
+		(property "Footprint" "Capacitor_SMD:C_0402_1005Metric"
 			(at 68.58 54.61 0)
 			(hide yes)
@@
 			)
 		)
-		(property "Footprint" ""
+		(property "Footprint" "Resistor_SMD:R_0402_1005Metric"
 			(at 129.54 54.61 0)
 			(hide yes)
@@
 			)
 		)
-		(property "Footprint" ""
+		(property "Footprint" "Resistor_SMD:R_0402_1005Metric"
 			(at 22.86 107.95 0)
 			(hide yes)
@@
 			)
 		)
-		(property "Footprint" ""
+		(property "Footprint" "Resistor_SMD:R_0402_1005Metric"
 			(at 185.42 107.95 0)
 			(hide yes)
@@
 			)
 		)
-		(property "Footprint" ""
+		(property "Footprint" "Capacitor_SMD:C_0402_1005Metric"
 			(at 170.18 54.61 0)
 			(hide yes)
@@
 			)
 		)
-		(property "Footprint" ""
+		(property "Footprint" "Resistor_SMD:R_0402_1005Metric"
 			(at 63.5 107.95 0)
 			(hide yes)
@@
 			)
 		)
-		(property "Footprint" ""
+		(property "Footprint" "RaceTracker:SODFL3517X110N"
 			(at 271.78 54.61 0)
 			(hide yes)
@@
 			)
 		)
-		(property "Footprint" ""
+		(property "Footprint" "RaceTracker:LED_0603_AK"
 			(at 104.14 107.95 0)
 			(hide yes)
@@
 			)
 		)
-		(property "Footprint" ""
+		(property "Footprint" "RaceTracker:ZED_F9P_LGA102"
 			(at 35.56 54.61 0)
 			(hide yes)
@@
 			)
 		)
-		(property "Footprint" ""
+		(property "Footprint" "Resistor_SMD:R_0402_1005Metric"
 			(at 83.82 107.95 0)
 			(hide yes)
@@
 			)
 		)
-		(property "Footprint" ""
+		(property "Footprint" "Resistor_SMD:R_0402_1005Metric"
 			(at 43.18 107.95 0)
 			(hide yes)
