File: RaceTracker.kicad_prj/Sensors_Storage.kicad_sch (KiCad schematic)
At the start: 19 parts, among them J10 MicroSD, J11 e-Paper (steckbar, Debug), U7 MPU-6050 (I2C 0x68)

Commit message: Zwei kritische Schaltplanfehler behoben
Power.kicad_sch: Vertikale GND-Busleitung bei x=20.32 (y=41.91–59.69)
entfernt, die J1.CC1 und J1.CC2 direkt auf GND kurzschloss. Die
Pull-Down-Widerstände R37/R38 (5,1 kΩ) waren damit elektrisch wirkungslos.
Ersetzt durch horizontale Verbindung (12.7, 41.91)→(20.32, 41.91) mit
eigenem GND-Symbol (#PWR042) für J1.GND.

Sensors_Storage.kicad_sch: Vertikale Leitung bei x=20.32 (y=50.8–77.47)
entfernt, die U7.AD0, U7.INT, U7.FSYNC und U7.CLKIN auf GND kurzschloss
und damit IMU_INT (PA10 des SAMD21) dauerhaft auf LOW zog. Ersetzt durch
drei kurze Leitungen mit separaten GND-Symbolen (#PWR100, #PWR101).

Co-Authored-By: Claude Sonnet 4.6 <noreply@anthropic.com>
Connections:
- net GND: no longer U7.11 (INT)
- new net IMU_INT: U7.11 (INT)
Changed lines of the file:
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@@
 	(wire
 		(pts
-			(xy 20.32 50.8) (xy 20.32 77.47)
+			(xy 13.97 50.8) (xy 20.32 50.8)
+		)
+		(stroke
+			(width 0)
+			(type default)
+		)
+	)
+	(wire
+		(pts
+			(xy 20.32 55.88) (xy 20.32 58.42)
+		)
+		(stroke
+			(width 0)
+			(type default)
+		)
+	)
+	(wire
+		(pts
+			(xy 13.97 58.42) (xy 20.32 58.42)
 		)
 		(stroke
@@
 					(unit 1)
 				)
+			)
+		)
+	)
+	(symbol
+		(lib_id "RaceTracker:GND")
+		(at 13.97 50.8 0)
+		(unit 1)
+		(body_style 1)
+		(exclude_from_sim no)
+		(in_bom no)
+		(on_board no)
+		(in_pos_files yes)
+		(dnp no)
+		(property "Reference" "#PWR100"
+			(at 13.97 57.8 0)
+			(hide yes)
+			(show_name no)
+			(do_not_autoplace no)
+			(effects
+				(font
+					(size 1.27 1.27)
+				)
+			)
+		)
+		(property "Value" "GND"
+			(at 4.97 50.8 0)
+			(show_name no)
+			(do_not_autoplace no)
+			(effects
+				(font
+					(size 1.4 1.4)
+				)
+			)
+		)
+		(property "Footprint" ""
+			(at 13.97 50.8 0)
+			(show_name no)
+			(do_not_autoplace no)
+			(effects
+				(font
+					(size 1.27 1.27)
+				)
+			)
+		)
+		(property "Datasheet" ""
+			(at 13.97 50.8 0)
+			(show_name no)
+			(do_not_autoplace no)
+			(effects
+				(font
+					(size 1.27 1.27)
+				)
+			)
+		)
+		(property "Description" ""
+			(at 13.97 50.8 0)
+			(show_name no)
+			(do_not_autoplace no)
+			(effects
+				(font
+					(size 1.27 1.27)
+				)
+			)
+		)
+		(pin "1"
+		)
+		(instances
+			(project "RaceTracker"
+				(path "/91b37a92-c006-41eb-be41-a2390c5c45b2/c38cb3c4-50cf-488f-b4da-82cd6a0246af"
+					(reference "#PWR100")
+					(unit 1)
+				)
+			)
+		)
+	)
+	(symbol
+		(lib_id "RaceTracker:GND")
+		(at 13.97 58.42 0)
+		(unit 1)
+		(body_style 1)
+		(exclude_from_sim no)
+		(in_bom no)
+		(on_board no)
+		(in_pos_files yes)
+		(dnp no)
+		(property "Reference" "#PWR101"
+			(at 13.97 65.42 0)
+			(hide yes)
+			(show_name no)
+			(do_not_autoplace no)
+			(effects
+				(font
+					(size 1.27 1.27)
+				)
+			)
+		)
+		(property "Value" "GND"
+			(at 4.97 58.42 0)
+			(show_name no)
+			(do_not_autoplace no)
+			(effects
+				(font
+					(size 1.4 1.4)
+				)
+			)
+		)
+		(property "Footprint" ""
+			(at 13.97 58.42 0)
+			(show_name no)
+			(do_not_autoplace no)
+			(effects
+				(font
+					(size 1.27 1.27)
+				)
+			)
+		)
+		(property "Datasheet" ""
+			(at 13.97 58.42 0)
+			(show_name no)
+			(do_not_autoplace no)
+			(effects
+				(font
+					(size 1.27 1.27)
+				)
+			)
+		)
+		(property "Description" ""
+			(at 13.97 58.42 0)
+			(show_name no)
+			(do_not_autoplace no)
+			(effects
+				(font
+					(size 1.27 1.27)
+				)
+			)
+		)
+		(pin "1"
+		)
+		(instances
+			(project "RaceTracker"
+				(path "/91b37a92-c006-41eb-be41-a2390c5c45b2/c38cb3c4-50cf-488f-b4da-82cd6a0246af"
+					(reference "#PWR101")
+					(unit 1)
+				)

Commit message: Footprints für GPS+Sensors_Storage: 132/132 Bauteile jetzt komplett
GPS-Blatt: SMA_EDGE, ML414H_COIN_CELL und ZED_F9P_LGA102 (bereits
vorhandene Custom-Footprints) verlinkt, Pad-Namen gegen Schaltplan-Pins
verifiziert. Restliche Passiva auf Standardbibliothek gemappt.

Sensors_Storage-Blatt: U7 (MPU-6050) auf KiCads eigene
Sensor_Motion:InvenSense_QFN-24_4x4mm_P0.5mm (exakt für diesen Chip
vorgesehen, nicht generisch geraten). J10 (MicroSD) auf
Connector_Card:microSD_HC_Molex_104031-0811 (Industriestandard-Teil).
J11 (e-Paper) auf 2,54mm-8-Pin-Stiftleiste, passend zum "steckbar"-Debug-
Anschluss von Waveshare-e-Paper-Modulen.

Damit haben alle 132 Bauteile im Projekt ein Footprint (vorher 1/132).
ERC weiterhin 0 Fehler/0 Warnungen, inklusive Footprint-Bibliotheksprüfung.

Co-Authored-By: Claude Sonnet 5 <noreply@anthropic.com>
Parts:
- C40, C41, C42, C44, C45: footprint (none) -> Capacitor_SMD:C_0402_1005Metric
- C43: footprint (none) -> Capacitor_SMD:C_0603_1608Metric
- DL10, DL11, DL12: footprint (none) -> RaceTracker:LED_0603_AK
- J10: footprint (none) -> Connector_Card:microSD_HC_Molex_104031-0811
- J11: footprint (none) -> Connector_PinHeader_2.54mm:PinHeader_1x08_P2.54mm_Vertical
- R40, R41, R42, R43, R44, R45, R46: footprint (none) -> Resistor_SMD:R_0402_1005Metric
- U7: footprint (none) -> Sensor_Motion:InvenSense_QFN-24_4x4mm_P0.5mm
Changed lines of the file:
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@@
 			)
 		)
-		(property "Footprint" ""
+		(property "Footprint" "Capacitor_SMD:C_0402_1005Metric"
 			(at 109.22 52.07 0)
 			(hide yes)
@@
 			)
 		)
-		(property "Footprint" ""
+		(property "Footprint" "Resistor_SMD:R_0402_1005Metric"
 			(at 236.22 52.07 0)
 			(hide yes)
@@
 			)
 		)
-		(property "Footprint" ""
+		(property "Footprint" "Resistor_SMD:R_0402_1005Metric"
 			(at 134.62 115.57 0)
 			(hide yes)
@@
 			)
 		)
-		(property "Footprint" ""
+		(property "Footprint" "Connector_PinHeader_2.54mm:PinHeader_1x08_P2.54mm_Vertical"
 			(at 35.56 115.57 0)
 			(hide yes)
@@
 			)
 		)
-		(property "Footprint" ""
+		(property "Footprint" "Resistor_SMD:R_0402_1005Metric"
 			(at 93.98 115.57 0)
 			(hide yes)
@@
 			)
 		)
-		(property "Footprint" ""
+		(property "Footprint" "Resistor_SMD:R_0402_1005Metric"
 			(at 276.86 52.07 0)
 			(hide yes)
@@
 			)
 		)
-		(property "Footprint" ""
+		(property "Footprint" "Capacitor_SMD:C_0402_1005Metric"
 			(at 53.34 115.57 0)
 			(hide yes)
@@
 			)
 		)
-		(property "Footprint" ""
+		(property "Footprint" "Connector_Card:microSD_HC_Molex_104031-0811"
 			(at 142.24 52.07 0)
 			(hide yes)
@@
 			)
 		)
-		(property "Footprint" ""
+		(property "Footprint" "Resistor_SMD:R_0402_1005Metric"
 			(at 175.26 52.07 0)
 			(hide yes)
@@
 			)
 		)
-		(property "Footprint" ""
+		(property "Footprint" "Capacitor_SMD:C_0402_1005Metric"
 			(at 68.58 52.07 0)
 			(hide yes)
@@
 			)
 		)
-		(property "Footprint" ""
+		(property "Footprint" "RaceTracker:LED_0603_AK"
 			(at 73.66 115.57 0)
 			(hide yes)
@@
 			)
 		)
-		(property "Footprint" ""
+		(property "Footprint" "Resistor_SMD:R_0402_1005Metric"
 			(at 175.26 115.57 0)
 			(hide yes)
@@
 			)
 		)
-		(property "Footprint" ""
+		(property "Footprint" "Resistor_SMD:R_0402_1005Metric"
 			(at 256.54 52.07 0)
 			(hide yes)
@@
 			)
 		)
-		(property "Footprint" ""
+		(property "Footprint" "Sensor_Motion:InvenSense_QFN-24_4x4mm_P0.5mm"
 			(at 35.56 52.07 0)
 			(hide yes)
@@
 			)
 		)
-		(property "Footprint" ""
+		(property "Footprint" "Capacitor_SMD:C_0402_1005Metric"
 			(at 88.9 52.07 0)
 			(hide yes)
@@
 			)
 		)
-		(property "Footprint" ""
+		(property "Footprint" "Capacitor_SMD:C_0603_1608Metric"
 			(at 195.58 52.07 0)
 			(hide yes)
@@
 			)
 		)
-		(property "Footprint" ""
+		(property "Footprint" "RaceTracker:LED_0603_AK"
 			(at 154.94 115.57 0)
 			(hide yes)
@@
 			)
 		)
-		(property "Footprint" ""
+		(property "Footprint" "Capacitor_SMD:C_0402_1005Metric"
 			(at 215.9 52.07 0)
 			(hide yes)
@@
 			)
 		)
-		(property "Footprint" ""
+		(property "Footprint" "RaceTracker:LED_0603_AK"
 			(at 114.3 115.57 0)
 			(hide yes)

Commit message: Sensors_Storage-Blatt gegen Datenblätter geprüft: C42 war 1000x zu groß
Gegen das offizielle InvenSense MPU-6000/6050 Product Specification
(Abschnitt 7.3, Bill of Materials for External Components) geprüft:

- C42 (Ladungspumpen-Kondensator an CPOUT, Pin 20): war 2u2 (2,2µF),
  Datenblatt verlangt exakt 2,2nF — Faktor-1000-Fehler behoben.
  Falscher Wert hätte die interne Ladungspumpe (versorgt die
  MEMS-Gyroskop-Oszillatoren) vermutlich funktionsunfähig gemacht.
- C41 (Regler-Filterkondensator an REGOUT, Pin 10, 100nF): korrekt,
  entspricht der Datenblattvorgabe von 0,1µF.
- AD0 auf GND → I2C-Adresse 0x68, stimmt mit der Schaltplan-Beschriftung
  überein.
- CLKIN/FSYNC auf GND: laut Datenblatt korrekt ("Connect to GND if
  unused").
- MicroSD (J10): DAT1/DAT2/CS/CARD_DET-Pullups (R40-R43) entsprechen
  dem empfohlenen SPI-Modus-Beschaltungsschema für SD-Karten.
- e-Paper (J11): vollständiger SPI-Signalsatz (VCC/GND/DIN/CLK/CS/DC/
  RST/BUSY) vorhanden und plausibel; exakte Pin-Reihenfolge hängt vom
  noch nicht gewählten konkreten Modul ab (offene BOM-Frage).

ERC weiterhin 0 Fehler/0 Warnungen.

Co-Authored-By: Claude Sonnet 5 <noreply@anthropic.com>
Parts:
- C42: value 2u2 (CPOUT) -> 2n2 (CPOUT)
Changed lines of the file:
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@@
 			)
 		)
-		(property "Value" "2u2 (CPOUT)"
+		(property "Value" "2n2 (CPOUT)"
 			(at 109.22 56.47 0)
 			(show_name no)
