File: v2-simple/kicad/RaceTracker_v2.kicad_sch (KiCad schematic)
At the start: 76 parts, among them J1 USB-C Sink, J10 MicroSD, J12 SWD-Programmierheader, J20 GPS 8p, J21 e-Paper (steckbar) 8p, J22 WiFi 8p, J7 LiPo, Q2 SIA817, Q3 2N7002, U1 D21G18, U5 BQ24195L, U6 AP2112K-3.3 -> +3V3, Y1 32768Hz

Commit message: v2-simple: echte Eagle-Symbolgrafik statt selbstgezeichneter Symbole
Alle MKR-referenz-abgeleiteten Bauteile (R/C/L/PTC-Passive, SAMD21, BQ24195L,
AP2112K-3.3, ESD-Diode, SIA817, 2N7002, PTS820-Taster, Kristall, LiPo-JST,
LED, Schottky-Diode) nutzen jetzt die per KiCad-Eagle-Import erzeugte
Original-Grafik aus der Arduino-MKR-WiFi-1010-Referenz statt der bisherigen
Generic-Symbole, auf Wunsch des Nutzers ("die sehen verschieden aus").

Bibliothek dazu neu unter reference/eagle/ (gemeinsam nutzbare Referenz,
analog zum ursprünglich vorgesehenen, aber nie angelegten reference/-Ordner).
Vor der Übernahme wurde jede Pin-NUMMER (nicht nur Anzahl) 1:1 gegen die
bereits ERC-geprüften v1-Symbole verglichen -- nur die Grafik ändert sich,
keine Elektrik. Custom-Bauteile ohne Eagle-Vorbild (SWD-Header, MicroSD,
e-Paper/GPS/WiFi-Stecker) und der bewusst abweichende USB-C-Stecker (Referenz
nutzt Micro-USB) bleiben unverändert.

Nebenbei zwei Bugs in der Geometrie-Extraktion gefunden und behoben:
- Sub-Unit-Suffix war auf "_1" hartkodiert; Eagle-Importe nutzen "_0"
  (SAMD21/SIA817 sind mehrteilige Symbole und blieben sonst leer)
- Referenz-/Werttext saß bei kleinen Eagle-Passiv-Symbolen auf dem eigenen
  Bauteilkörper (deren Standard-Textabstand ist knapper als bei den alten
  Symbolen) -- Textposition wird jetzt aus der tatsächlichen Bounding-Box
  berechnet statt aus der Symbol-Vorgabe übernommen.

Kollisionsprüfung (Körper, eigener und fremder Text) weiterhin 0 Treffer;
kicad-cli erc/netlist/pdf zur Kontrolle verifiziert (76 Bauteile vollständig
in der Netzliste, keine unaufgelösten Pin-Typen mehr).

Co-Authored-By: Claude Sonnet 5 <noreply@anthropic.com>
Parts:
- removed C1: 4n7, Capacitor_SMD:C_0805_2012Metric, symbol RaceTracker:C_GENERIC
- removed C12, C13, C19, C20: 10u, Capacitor_SMD:C_0603_1608Metric, symbol RaceTracker:C_GENERIC
- removed C14, C22, C25, C26, C32: 1u, Capacitor_SMD:C_0402_1005Metric, symbol RaceTracker:C_GENERIC
- removed C15: 47n, Capacitor_SMD:C_0402_1005Metric, symbol RaceTracker:C_GENERIC
- removed C16, C5: 4u7, Capacitor_SMD:C_0402_1005Metric, symbol RaceTracker:C_GENERIC
- removed C17, C18, C2, C21, C23, C24, C6, C7: 100n, Capacitor_SMD:C_0402_1005Metric, symbol RaceTracker:C_GENERIC
- removed C27: 4u7, Capacitor_SMD:C_0603_1608Metric, symbol RaceTracker:C_GENERIC
- removed C3, C4: 20p, Capacitor_SMD:C_0402_1005Metric, symbol RaceTracker:C_GENERIC
- removed C43: 10u (SD), Capacitor_SMD:C_0603_1608Metric, symbol RaceTracker:C_GENERIC
- removed C44: 100n (SD), Capacitor_SMD:C_0402_1005Metric, symbol RaceTracker:C_GENERIC
- removed D1: PRTR5V, RaceTracker:SOT143B_4N, symbol RaceTracker:ESD_PRTR5V0U2X
- removed D2, D3: PMEG6020, RaceTracker:SODFL3517X110N, symbol RaceTracker:DIODE_AC
- removed DL10: gruen GPS-Fix, RaceTracker:LED_0603_AK, symbol RaceTracker:LED_AC
- removed DL11: blau Aufnahme, RaceTracker:LED_0603_AK, symbol RaceTracker:LED_AC
- removed DL12: rot Fehler, RaceTracker:LED_0603_AK, symbol RaceTracker:LED_AC
- removed DL2: orange Laden, RaceTracker:LED_0603_AK, symbol RaceTracker:LED_AC
- removed DL3: gruen USB, RaceTracker:LED_0603_AK, symbol RaceTracker:LED_AC
- removed F1, F2: MFFSMF050, Fuse:Fuse_0603_1608Metric, symbol RaceTracker:PTC_GENERIC
- removed J7: LiPo, RaceTracker:JST_S2B_PH_SM4_TB, symbol RaceTracker:CONN_JST_PH_2P
- removed L2: 2u2, RaceTracker:SRP4020, symbol RaceTracker:L_GENERIC
- removed L3: BLM18PG471, Inductor_SMD:L_0603_1608Metric, symbol RaceTracker:FERRITE_GENERIC
- removed PB1: Reset, RaceTracker:PTS820_NO_HOLES, symbol RaceTracker:SW_PUSH_PTS820
- removed Q2: SIA817, RaceTracker:SON65P205X205X75-8N-MWSD, symbol RaceTracker:MOSFET_PMOS_DIODE_SIA817
- removed Q3: 2N7002, RaceTracker:SOTFL50P160X78-3, symbol RaceTracker:MOSFET_NCH_SOT523
- removed R1: 1M, Resistor_SMD:R_0402_1005Metric, symbol RaceTracker:R_GENERIC
- removed R10, R19: 100k, Resistor_SMD:R_0402_1005Metric, symbol RaceTracker:R_GENERIC
- removed R13, R14: 4k7, Resistor_SMD:R_0402_1005Metric, symbol RaceTracker:R_GENERIC
- removed R23, R28, R3, R6: 330R, Resistor_SMD:R_0402_1005Metric, symbol RaceTracker:R_GENERIC
- removed R24, R25, R26, R29, R5: 10k, Resistor_SMD:R_0402_1005Metric, symbol RaceTracker:R_GENERIC
- removed R27: 390R, Resistor_SMD:R_0402_1005Metric, symbol RaceTracker:R_GENERIC
- removed R30: 5k49, Resistor_SMD:R_0402_1005Metric, symbol RaceTracker:R_GENERIC
- removed R37: 5k1 CC1, Resistor_SMD:R_0402_1005Metric, symbol RaceTracker:R_GENERIC
- removed R38: 5k1 CC2, Resistor_SMD:R_0402_1005Metric, symbol RaceTracker:R_GENERIC
- removed R40: 10k (SD_CS Pullup), Resistor_SMD:R_0402_1005Metric, symbol RaceTracker:R_GENERIC
- removed R44, R45, R46: 1k, Resistor_SMD:R_0402_1005Metric, symbol RaceTracker:R_GENERIC
- removed R8: 330k, Resistor_SMD:R_0402_1005Metric, symbol RaceTracker:R_GENERIC
- removed R9: 1M2, Resistor_SMD:R_0402_1005Metric, symbol RaceTracker:R_GENERIC
- removed U1: D21G18, RaceTracker:QFN48_SAMD21G18A, symbol RaceTracker:SAMD21G18A_QFN48
- removed U5: BQ24195L, RaceTracker:QFN24_BQ24195L, symbol RaceTracker:BQ24195L_QFN24
- removed U6: AP2112K-3.3 -> +3V3, RaceTracker:SOT25, symbol RaceTracker:AP2112K_33_SOT25
- removed Y1: 32768Hz, RaceTracker:ABS07_CRYSTAL, symbol RaceTracker:CRYSTAL_32K768
- added C1: 4n7, Capacitor_SMD:C_0805_2012Metric, symbol RaceTracker:C-0805
- added C12, C13, C19, C20: 10u, Capacitor_SMD:C_0603_1608Metric, symbol RaceTracker:C-0603
- added C14, C22, C25, C26, C32: 1u, Capacitor_SMD:C_0402_1005Metric, symbol RaceTracker:C-0402
- added C15: 47n, Capacitor_SMD:C_0402_1005Metric, symbol RaceTracker:C-0402
- added C16, C5: 4u7, Capacitor_SMD:C_0402_1005Metric, symbol RaceTracker:C-0402
- added C17, C18, C2, C21, C23, C24, C6, C7: 100n, Capacitor_SMD:C_0402_1005Metric, symbol RaceTracker:C-0402
- added C27: 4u7, Capacitor_SMD:C_0603_1608Metric, symbol RaceTracker:C-0603
- added C3, C4: 20p, Capacitor_SMD:C_0402_1005Metric, symbol RaceTracker:C-0402
- added C43: 10u (SD), Capacitor_SMD:C_0603_1608Metric, symbol RaceTracker:C-0603
- added C44: 100n (SD), Capacitor_SMD:C_0402_1005Metric, symbol RaceTracker:C-0402
- added D1: PRTR5V, RaceTracker:SOT143B_4N, symbol RaceTracker:PRTR5V0U2X,215
- added D2, D3: PMEG6020, RaceTracker:SODFL3517X110N, symbol RaceTracker:PMEG6020AELRX
- added DL10: gruen GPS-Fix, RaceTracker:LED_0603_AK, symbol RaceTracker:LED-0603
- added DL11: blau Aufnahme, RaceTracker:LED_0603_AK, symbol RaceTracker:LED-0603
- added DL12: rot Fehler, RaceTracker:LED_0603_AK, symbol RaceTracker:LED-0603
- added DL2: orange Laden, RaceTracker:LED_0603_AK, symbol RaceTracker:LED-0603
- added DL3: gruen USB, RaceTracker:LED_0603_AK, symbol RaceTracker:LED-0603
- added F1, F2: MFFSMF050, Fuse:Fuse_0603_1608Metric, symbol RaceTracker:PTC
- added J7: LiPo, RaceTracker:JST_S2B_PH_SM4_TB, symbol RaceTracker:BATTERY
- added L2: 2u2, RaceTracker:SRP4020, symbol RaceTracker:LSRP
- added L3: BLM18PG471, Inductor_SMD:L_0603_1608Metric, symbol RaceTracker:FERRITE0603
- added PB1: Reset, RaceTracker:PTS820_NO_HOLES, symbol RaceTracker:TACTILE1PTS820-NH
- added Q2: SIA817, RaceTracker:SON65P205X205X75-8N-MWSD, symbol RaceTracker:SIA817EDJ
- added Q3: 2N7002, RaceTracker:SOTFL50P160X78-3, symbol RaceTracker:2N7002T-SOT523
- added R1: 1M, Resistor_SMD:R_0402_1005Metric, symbol RaceTracker:R-0402
- added R10, R19: 100k, Resistor_SMD:R_0402_1005Metric, symbol RaceTracker:R-0402
- added R13, R14: 4k7, Resistor_SMD:R_0402_1005Metric, symbol RaceTracker:R-0402
- added R23, R28, R3, R6: 330R, Resistor_SMD:R_0402_1005Metric, symbol RaceTracker:R-0402
- added R24, R25, R26, R29, R5: 10k, Resistor_SMD:R_0402_1005Metric, symbol RaceTracker:R-0402
- added R27: 390R, Resistor_SMD:R_0402_1005Metric, symbol RaceTracker:R-0402
- added R30: 5k49, Resistor_SMD:R_0402_1005Metric, symbol RaceTracker:R-0402
- added R37: 5k1 CC1, Resistor_SMD:R_0402_1005Metric, symbol RaceTracker:R-0402
- added R38: 5k1 CC2, Resistor_SMD:R_0402_1005Metric, symbol RaceTracker:R-0402
- added R40: 10k (SD_CS Pullup), Resistor_SMD:R_0402_1005Metric, symbol RaceTracker:R-0402
- added R44, R45, R46: 1k, Resistor_SMD:R_0402_1005Metric, symbol RaceTracker:R-0402
- added R8: 330k, Resistor_SMD:R_0402_1005Metric, symbol RaceTracker:R-0402
- added R9: 1M2, Resistor_SMD:R_0402_1005Metric, symbol RaceTracker:R-0402
- added U1: D21G18, RaceTracker:QFN48_SAMD21G18A, symbol RaceTracker:ATSAMD21G18A-48QFN
- added U5: BQ24195L, RaceTracker:QFN24_BQ24195L, symbol RaceTracker:BQ24195QFN-24
- added U6: AP2112K-3.3 -> +3V3, RaceTracker:SOT25, symbol RaceTracker:AP2112K-3.3
- added Y1: 32768Hz, RaceTracker:ABS07_CRYSTAL, symbol RaceTracker:32.768KHZ
Connections:
- new net: J7.3 (SH), J7.4 (SH)
- new net: PB1.1 (3), PB1.2 (3), PB1.3, PB1.4 (3)
- new net: U5.1 (VBUS), U5.24 (VBUS)
- new net: U5.13 (BAT), U5.14 (BAT)
- new net: U5.15 (SYS), U5.16 (SYS)
- new net: U5.17 (PGND), U5.18 (PGND)
- new net: U5.19 (SW), U5.20 (SW)
- new net: Q2.D, Q2.D2 (D)
- new net: Q2.K (C), Q2.K2 (C)
