File: v2-simple/kicad/RaceTracker_v2.kicad_sch (KiCad schematic)
At the start: 76 parts, among them J1 USB-C Sink, J10 MicroSD, J12 SWD-Programmierheader, J20 GPS 8p, J21 e-Paper (steckbar) 8p, J22 WiFi 8p, J7 LiPo, Q2 SIA817, Q3 2N7002, U1 D21G18, U5 BQ24195L, U6 AP2112K-3.3 -> +3V3, Y1 32768Hz

Commit message: v2-simple: fehlende Schutz-/Pullup-Bauteile ergänzt (D4, C34, R2, R21, R43)
Teileabgleich gegen v1 zeigte 5 echte Lücken unabhängig von der bewussten
GPS/NINA/MPU-Reduktion: USB-VBUS-ESD-Schutz (D4) und -Entkopplung (C34) an
J1, SWD-Reset-Schutzwiderstand (R2) an J12, OTG-Erkennungs-Pullup (R21) am
Q3-Gate, SD-Card-Detect-Pullup (R43) an J10. Alle 5 existieren bereits
ERC-geprüft in v1 und wurden über die bestehende extract_v1.py ->
map_eagle_symbols.py -> gen_symbols_v2.py -> build_sheet_v2.py Pipeline neu
gezogen (Werte/Footprints 1:1 aus v1, Eagle-Symbolgrafik erhalten). Keine
Kollisionen, SVG-Export geprüft.
Parts:
- added C34: 1uF VBUS decoupling, Capacitor_SMD:C_0402_1005Metric, symbol RaceTracker:C-0402
- added D4: PESD5V0S1BA TVS VBUS, Diode_SMD:D_SOD-323, symbol RaceTracker:PMEG6020AELRX
- added R2: 39R SWD nRESET, Resistor_SMD:R_0402_1005Metric, symbol RaceTracker:R-0402
- added R21: 10k, Resistor_SMD:R_0402_1005Metric, symbol RaceTracker:R-0402
- added R43: 10k (Card-Detect), Resistor_SMD:R_0402_1005Metric, symbol RaceTracker:R-0402

Commit message: v2-simple: kompletten Schaltplan verdrahtet, R4 als 6. fehlender SWD-Pull-up ergänzt
Netzliste (netmap_v2.json) aus der echten kicad-cli-Netlist von v1 abgeleitet
(GPS.kicad_sch ausgeschlossen, GPS-Modul bewusst nicht bestückt -- Anschluss
folgt später extern über J20). Neues Skript wire_v2.py berechnet jede
Pin-Position aus Instanz-Platzierung + Symbol-Pin-Geometrie und setzt lokale
Labels, No-Connect-Marker und 8 PWR_FLAGs (GND/VBAT/+5V/CHG_VBUS für Netze
ganz ohne power_out-Pin; +3V3/+3V8/VDDANA/VDDCORE zusätzlich nach echter ERC).
J20 (GPS) bekommt nur SDA/SCL/3V3/GND (geteilter I2C-Bus wie ZED-F9P in v1);
J22 (WiFi) übernimmt die SERCOM-Pins von NINA-W102 in v1 (PB22/PB23 UART,
PA14/PA15 RTS/CTS); J21 (e-Paper) übernimmt 1:1 die Netze von v1s J11.

Beim Bau des Pin-Positions-Codes einen Analyzer-Bug entdeckt: kicad-happy
zeigte für die SWCLK/SWDIO-Pins des Eagle-Mehrfachsymbols (ATSAMD21G18A)
fälschlich "+3V3" statt der echten Netze -- über die echte kicad-cli-Netlist
aufgefallen, dabei R4 (SWCLK-Pull-up) als sechsten fehlenden Schutzwiderstand
gefunden (war in der ersten Teileprüfung fälschlich als "totes Bauteil"
eingestuft, weil beide Analyzer-Pins auf "+3V3" zeigten).

Label-Platzierung: jedes Label sitzt am Ende eines kurzen (6.5mm) Stubs statt
direkt am Pin -- sonst kollidiert der Text bei senkrecht bepinnten Bauteilen
mit dem Referenz-/Werttext, den build_sheet_v2.py schon über/unter dem
Bauteilkörper zeichnet (computational per Text-Bounding-Box-Check gefunden,
82 Fälle). GAP_INTRA/SUBUNIT_GAP erhöht (18/20mm) für mehr Label-Freiraum.
Eine zusätzliche Direktverdrahtung eng benachbarter gleichnamiger Pins wurde
erwogen, aber wieder verworfen: sie erzeugte einen echten GND<->+3V3- bzw.
CHG_TS<->CHG_REGN-Kurzschluss, weil die Gerade zum nächsten gleichnamigen
Pin am näher liegenden, andersnetzigen Pin eines dritten Bauteils vorbeilief.

Verifikation: kicad-cli sch export netlist stimmt für alle 60 Netze exakt
mit der beabsichtigten Verkabelung überein; kic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
Parts:
- added R4: 1k, Resistor_SMD:R_0402_1005Metric, symbol RaceTracker:R-0402
Connections:
- net LED_REC: now reaches R45.1
- net LED_REC: now also U1.31 (PA22)
- net DL11_A: now reaches R45.2
- net DL11_A: now also DL11.A
- net VUSB1: now reaches D3.A
- net VUSB1: now also C12.1, C13.1, U5.23 (PMID)
- net +5V: now reaches D3.C
- net +5V: now also D1.4, F1.2, Q2.D, Q2.D2 (D)
- net PA03_VREFA: now reaches C7.1
- net PA03_VREFA: now also C5.1, U1.4 (PA03)
- net GND: now reaches C7.2
- net GND: now also C1.2, C12.2, C13.2, C14.2, C16.2, C17.2, C18.2, C19.2, C2.2, C20.2, C21.2, C22.2, C23.2, C24.2, C25.2, C26.2, C27.2, C3.1, C32.2, C34.2, C4.1, C43.2, C44.2, C5.2, C6.2, D2.A, D4.A, DL10.C, DL11.C, DL12.C, DL3.C, J1.A1 (GND), J1.A12 (GND), J1.B1 (GND), J1.B12 (GND), J1.SH (SHIELD), J10.10 (SHIELD), J10.6 (VSS), J12.5 (GND), J20.8 (GND), J21.8 (GND), J22.8 (GND), J7.2, J7.3 (SH), J7.4 (SH), PB1.1 (3), PB1.2 (3), PB1.3, PB1.4 (3), PB1.5 (1), Q3.S, R1.1, R10.2, R19.1, R25.1, R28.2, R29.1, R37.2, R38.2, R9.1, U1.18 (GND), U1.35 (GND), U1.42 (GND), U1.49 (EP), U1.5 (GNDANA), U5.17 (PGND), U5.18 (PGND), U5.25 (TH), U6.2 (GND/ADJ)
- net +3V3: now reaches R26.1
- net +3V3: now also C17.1, C18.1, C21.1, C24.1, C26.1, C43.1, C44.1, J10.4 (VDD), J12.4 (+3V3), J20.1 (3V3), J21.1 (VCC), J22.1 (3V3), L3.1, R13.2, R14.2, R21.1, R24.1, R40.2, R43.2, R5.2, U1.17 (VDDIO), U1.36 (VDDIO), U1.44 (VDDIN), U6.5 (OUT), R4.2
- net CHG_OTG: now reaches R26.2
- net CHG_OTG: now also Q3.D, U5.8 (OTG)
- net VDDANA: now reaches C23.1
- net VDDANA: now also C27.1, L3.2, U1.6 (VDDANA)
- net USBC_VBUS: now reaches D4.C
- net USBC_VBUS: now also C34.1, F1.1, J1.A4 (VBUS), J1.A9 (VBUS), J1.B4 (VBUS), J1.B9 (VBUS)
- net I2C_SCL: now reaches R13.1
- net I2C_SCL: now also J20.3 (SCL), U1.14 (PA09), U5.5 (SCL)
- net CHG_BTST: now reaches C15.1
- net CHG_BTST: now also U5.21 (BTST)
- net CHG_SW: now reaches C15.2
- net CHG_SW: now also L2.1, U5.19 (SW), U5.20 (SW)
- net SPI_MOSI: now reaches J21.2 (DIN)
- net SPI_MOSI: now also J10.3 (CMD (MOSI)), U1.25 (PA16)
- net SPI_SCK: now reaches J21.3 (CLK)
- net SPI_SCK: now also J10.5 (CLK (SCK)), U1.26 (PA17)
- net EPD_CS: now reaches J21.4 (CS)
- net EPD_CS: now also U1.11 (PA06)
- net EPD_DC: now reaches J21.5 (DC)
- net EPD_DC: now also U1.10 (PA05)
- net EPD_RST: now reaches J21.6 (RST)
- net EPD_RST: now also U1.9 (PA04)
- net EPD_BUSY: now reaches J21.7 (BUSY)
- net EPD_BUSY: now also U1.3 (PA02)
- net PB09_FILT: now reaches R8.1
- net PB09_FILT: now also C6.1, R9.2, U1.8 (PB09)
- net VBAT: now reaches R8.2
- net VBAT: now also D2.C, F2.2, U5.13 (BAT), U5.14 (BAT)
- net XIN32: now reaches U1.1 (PA00/XIN32)
- net XIN32: now also C3.2, Y1.2
- net SD_CS: now reaches U1.12 (PA07)
- net SD_CS: now also J10.2 (CD/DAT3 (CS)), R40.1
- net I2C_SDA: now reaches U1.13 (PA08)
- net I2C_SDA: now also J20.2 (SDA), R14.1, U5.6 (SDA)
- net XOUT32: now reaches U1.2 (PA01/XOUT32)
- net XOUT32: now also C4.2, Y1.1
- net SD_CD: now reaches U1.20 (PB11)
- net SD_CD: now also J10.9 (CARD_DET), R43.1
- net WIFI_CTS: now reaches U1.23 (PA14)
- net WIFI_CTS: now also J22.5 (CTS)
- net WIFI_RTS: now reaches U1.24 (PA15)
- net WIFI_RTS: now also J22.4 (RTS)
- net PA18_OTG: now reaches U1.27 (PA18)
- net PA18_OTG: now also Q3.G, R21.2
- net SPI_MISO: now reaches U1.28 (PA19)
- net SPI_MISO: now also J10.7 (DAT0 (MISO))
- net LED_FIX: now reaches U1.30 (PA21)
- net LED_FIX: now also R44.1
- net LED_ERR: now reaches U1.32 (PA23)
- net LED_ERR: now also R46.1
- net USB_N: now reaches U1.33 (PA24/USB_DM)
- net USB_N: now also D1.3, J1.A7 (D-), J1.B7 (D-)
- net USB_P: now reaches U1.34 (PA25/USB_DP)
- net USB_P: now also D1.2, J1.A6 (D+), J1.B6 (D+)
- net PB22_S5_TX: now reaches U1.37 (PB22)
- net PB22_S5_TX: now also J22.3 (RX)
- net PB23_S5_RX: now reaches U1.38 (PB23)
- net PB23_S5_RX: now also J22.2 (TX)
- net RESETN: now reaches U1.40 (RESETN)
- net RESETN: now also C2.1, R2.2, R3.2, R5.1, R6.1
- net PA30_SWCLK: now reaches U1.45 (PA30/SWCLK)
- net PA30_SWCLK: now also J12.1 (SWCLK), R4.1
- net PA31_SWDIO: now reaches U1.46 (PA31/SWDIO)
- net PA31_SWDIO: now also J12.2 (SWDIO)
- net PB08_NC: now reaches U1.7 (PB08)
- net PB08_NC: now also R10.1
- net +3V8: now reaches C22.1
- net +3V8: now also C19.1, C20.1, C32.1, L2.2, R23.2, U5.15 (SYS), U5.16 (SYS), U6.1 (IN), U6.3 (EN)
- net USBC_CC1: now reaches J1.A5 (CC1)
- net USBC_CC1: now also R37.1
- net USBC_CC2: now reaches J1.B5 (CC2)
- net USBC_CC2: now also R38.1
- net CHG_ILIM: now reaches R28.1
- net CHG_ILIM: now also U5.10 (ILIM)
- net DL2_A: now reaches R23.1
- net DL2_A: now also DL2.A
- net D1_IO1: now reaches C1.1
- net D1_IO1: now also D1.1, R1.2
- net DL12_A: now reaches DL12.A
- net DL12_A: now also R46.2
- net VDDCORE: now reaches U1.43 (VDDCORE)
- net VDDCORE: now also C25.1
- net VIN: now reaches R19.2
- net VIN: now also Q2.A, Q2.G
- net CHG_VBUS: now reaches U5.1 (VBUS), U5.24 (VBUS)
- net CHG_VBUS: now also C14.1, Q2.K (C), Q2.K2 (C), Q2.S, R27.2
- net CHG_TS: now reaches U5.11 (TS1)
- net CHG_TS: now also R29.2, R30.2, U5.12 (TS2)
- net CHG_REGN: now reaches U5.22 (REGN)
- net CHG_REGN: now also C16.1, R30.1
- net CHG_STAT: now reaches U5.4 (STAT)
- net CHG_STAT: now also DL2.C
- net CHG_INT: now reaches U5.7 (INT)
- net CHG_INT: now also R24.2
- net CHG_CE: now reaches U5.9 (CE)
- net CHG_CE: now also R25.2
- net SWD_NRESET: now reaches J12.3 (nRESET)
- net SWD_NRESET: now also R2.1
- net RESET_SW_B: now reaches R3.1
- net RESET_SW_B: now also PB1.6 (2)
- net DL3_A: now reaches DL3.A
- net DL3_A: now also R27.1
- net DL10_A: now reaches DL10.A
- net DL10_A: now also R44.2
- net BATT_PLUS: now reaches F2.1
- net BATT_PLUS: now also J7.1
- no-connect marks 0 -> 23
