File: RaceTracker.kicad_prj/V3 ESP32/New Version with WROOM/New Version with WROOM.kicad_sch (KiCad schematic)
At the start: 39 parts, among them J1 USB-C, J2 Battery, J3 Qwiic GPS (I2C), J4 microSD, J5 UART Debug, SW1 PWR, SW2 RESET, SW3 BOOT, U1 ESP32-S3-WROOM-1-N8, U2 MCP73831T-2ACI/OT, U3 AP2112K-3.3

Commit message: V3: PCB-Footprint-Platzierung (kein Routing) + Widerstand-Footprint-Fix
- build_sch.py: generische "R" Bauteile hatten kein Footprint gesetzt
  (PART_LIB-Default war None) -- auf R_0603_1608Metric korrigiert.
- Neue PCB unter RaceTracker.kicad_prj/V3 ESP32/New Version with WROOM/:
  70x97mm, alle 39 Footprints platziert via tools/build_pcb.py (pcbnew-
  Python-Scripting) + tools/layout.py (Shelf-Packer mit real gemessenen
  Courtyard-Bounding-Boxen aus tools/fp_bbox.py, nicht geschaetzt --
  der erste Versuch mit Wunschkoordinaten ergab 43 DRC-Fehler).
  U1 um 90 Grad gedreht, damit die im offiziellen Footprint bereits
  enthaltene Antennen-Keepout-Zone zum linken Rand zeigt statt die
  komplette Oberkante zu blockieren.
- kicad-cli pcb drc: 0 Fehler (min_through_hole_diameter auf 0.2mm
  gelockert -- passt zum EPAD-Stitching-Via-Muster des offiziellen
  ESP32-S3-WROOM-1 Footprints), 104 unverbundene Punkte (erwartet,
  kein Routing wie angefragt).
- tools/pdn_check.py: ngspice-AC-Sweep der 3V3-Entkopplung gegen ein
  Ziel-Impedanzbudget aus dem echten Datenblatt-Peak (355mA WiFi-TX,
  Tabelle 6-4) und VDD33-Toleranz (Tabelle 6-2) -- besteht bei
  realistischem 150mV-Budget komfortabel.
Parts:
- R1, R10, R11, R12, R13, R14, R2, R3, R4, R5, R6, R7, R8, R9: footprint (none) -> Resistor_SMD:R_0603_1608Metric
Changed lines of the file:
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@@
 			(effects (font (size 1.27 1.27)))
 		)
-		(property "Footprint" ""
+		(property "Footprint" "Resistor_SMD:R_0603_1608Metric"
 			(at 204.47 123.19 0)
 			(effects (font (size 1.27 1.27)) hide)
@@
 			(effects (font (size 1.27 1.27)))
 		)
-		(property "Footprint" ""
+		(property "Footprint" "Resistor_SMD:R_0603_1608Metric"
 			(at 190.5 128.27 0)
 			(effects (font (size 1.27 1.27)) hide)
@@
 			(effects (font (size 1.27 1.27)))
 		)
-		(property "Footprint" ""
+		(property "Footprint" "Resistor_SMD:R_0603_1608Metric"
 			(at 203.2 148.59 0)
 			(effects (font (size 1.27 1.27)) hide)
@@
 			(effects (font (size 1.27 1.27)))
 		)
-		(property "Footprint" ""
+		(property "Footprint" "Resistor_SMD:R_0603_1608Metric"
 			(at 187.96 151.13 0)
 			(effects (font (size 1.27 1.27)) hide)
@@
 			(effects (font (size 1.27 1.27)))
 		)
-		(property "Footprint" ""
+		(property "Footprint" "Resistor_SMD:R_0603_1608Metric"
 			(at 195.58 153.67 0)
 			(effects (font (size 1.27 1.27)) hide)
@@
 			(effects (font (size 1.27 1.27)))
 		)
-		(property "Footprint" ""
+		(property "Footprint" "Resistor_SMD:R_0603_1608Metric"
 			(at 208.28 161.29 0)
 			(effects (font (size 1.27 1.27)) hide)
@@
 			(effects (font (size 1.27 1.27)))
 		)
-		(property "Footprint" ""
+		(property "Footprint" "Resistor_SMD:R_0603_1608Metric"
 			(at 180.34 163.83 0)
 			(effects (font (size 1.27 1.27)) hide)
@@
 			(effects (font (size 1.27 1.27)))
 		)
-		(property "Footprint" ""
+		(property "Footprint" "Resistor_SMD:R_0603_1608Metric"
 			(at 364.49 88.9 0)
 			(effects (font (size 1.27 1.27)) hide)
@@
 			(effects (font (size 1.27 1.27)))
 		)
-		(property "Footprint" ""
+		(property "Footprint" "Resistor_SMD:R_0603_1608Metric"
 			(at 374.65 91.44 0)
 			(effects (font (size 1.27 1.27)) hide)
@@
 			(effects (font (size 1.27 1.27)))
 		)
-		(property "Footprint" ""
+		(property "Footprint" "Resistor_SMD:R_0603_1608Metric"
 			(at 299.72 148.59 0)
 			(effects (font (size 1.27 1.27)) hide)
@@
 			(effects (font (size 1.27 1.27)))
 		)
-		(property "Footprint" ""
+		(property "Footprint" "Resistor_SMD:R_0603_1608Metric"
 			(at 284.48 162.56 0)
 			(effects (font (size 1.27 1.27)) hide)
@@
 			(effects (font (size 1.27 1.27)))
 		)
-		(property "Footprint" ""
+		(property "Footprint" "Resistor_SMD:R_0603_1608Metric"
 			(at 347.98 190.5 0)
 			(effects (font (size 1.27 1.27)) hide)
@@
 			(effects (font (size 1.27 1.27)))
 		)
-		(property "Footprint" ""
+		(property "Footprint" "Resistor_SMD:R_0603_1608Metric"
 			(at 330.2 210.82 0)
 			(effects (font (size 1.27 1.27)) hide)
@@
 			(effects (font (size 1.27 1.27)))
 		)
-		(property "Footprint" ""
+		(property "Footprint" "Resistor_SMD:R_0603_1608Metric"
 			(at 330.2 218.44 0)
 			(effects (font (size 1.27 1.27)) hide)
