File: RaceTracker.kicad_prj/V3 ESP32/RaceTracker_v3/RaceTracker_v3.kicad_sch (KiCad schematic)
At the start: 39 parts, among them J1 USB-C, J2 Battery, J3 Qwiic GPS (I2C), J4 microSD, J5 UART Debug, SW1 PWR, SW2 RESET, SW3 BOOT, U1 ESP32-S3-WROOM-1-N8, U2 MCP73831T-2ACI/OT, U3 AP2112K-3.3

Commit message: V3: C2 (MCP73831 VDD-Entkopplung) von 1uF auf 4.7uF korrigiert
Datenblatt-Review aller Bauteile gegen die jeweilige typische Beschaltung
(MCP73831, AP2112K-3.3, USBLC6-2SC6, PESD5V0S1UL real heruntergeladen und
gegengeprueft). Einziger echter Fund: MCP73831 Abschnitt 3.1 verlangt am
VDD-Pin explizit "Bypass to VSS with a minimum of 4.7 uF" -- C2 hatte nur
1uF. VBAT-seitige Entkopplung (C3=4.7uF) stimmte bereits exakt. AP2112K-3.3
(1uF/1uF), USBLC6-2SC6 (keine externen Bauteile noetig) und PESD5V0S1UL
(Polaritaet K->VBUS, A->GND) bestaetigt korrekt.

ERC 0/0, DRC 0 Fehler nach dem Fix weiterhin bestaetigt.
Parts:
- C2: value 1uF -> 4.7uF
Changed lines of the file:
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@@
 			(effects (font (size 1.27 1.27)))
 		)
-		(property "Value" "1uF"
+		(property "Value" "4.7uF"
 			(at 314.96 144.2 0)
 			(effects (font (size 1.27 1.27)))
