File: RaceTracker.kicad_prj/V3 ESP32/RaceTracker_v3/RaceTracker_v3.kicad_pcb (KiCad board)
At the start: 4 copper layers, 56 x 65.5 mm, 49 parts, among them J1 USB-C, J2 Battery, J3 Qwiic GPS (I2C), J4 microSD, J5 UART Debug, J6 e-Paper (steckbar) 8p, SW1 PWR, SW2 RESET, SW3 BOOT, U1 ESP32-S3-WROOM-1-N8, U2 MCP73831T-2ACI/OT, U3 AP2112K-3.3, U4 WSEN-ISDS

Commit message: V3: redundante Vias auf J3s PTH-Pads entfernt
J3 (PTH-Pinheader) verbindet ueber die Pad-Bohrung schon alle Kupferlagen
inkl. GND-/+3V3-Ebene - zwei Stitching-Vias saßen exakt auf den Pad-Loechern
(pin1/pin2), doppelte Bohrung an derselben Stelle, DRC holes_co_located.
Entfernt, analog zum gleichen Fund bei DBG_TXD0/EPD_RST vorhin.

Verifiziert: kicad-cli pcb drc --severity-all -> 0 Errors (nur die 5
erwarteten lib_footprint_mismatch-Warnings), 0 offene Verbindungen
(User hat das Routing inzwischen fertiggestellt). ERC weiterhin 0/0.

Co-Authored-By: Claude Sonnet 5 <noreply@anthropic.com>
Routing:
- net /I2C_SDA: track 53.9 -> 57.8 mm, vias 4 -> 3
- net /I2C_SCL: track 49.5 -> 53.2 mm, vias 4 -> 3
- net /GND: vias 40 -> 39
- net /+3V3: vias 22 -> 21
Changed lines of the file:
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@@
-	)
-	(via
-		(at 50.06 74.58)
-		(size 0.6)
-		(drill 0.3)
-		(layers "F.Cu" "B.Cu")
-		(net "/GND")
 	)
 	(via
@@
 	)
 	(via
-		(at 50.179099 75.830225)
-		(size 0.6)
-		(drill 0.3)
-		(layers "F.Cu" "B.Cu")
-		(net "/+3V3")
-	)
-	(via
 		(at 54.5 79)
 		(size 0.6)
@@
 	)
 	(via
-		(at 49.5 77)
-		(size 0.6)
-		(drill 0.3)
-		(layers "F.Cu" "B.Cu")
-		(net "/I2C_SDA")
-	)
-	(via
 		(at 91.295603 66.352)
 		(size 0.6)
@@
 	)
 	(segment
+		(start 52.08 77)
+		(end 47.5 81.58)
+		(width 0.2)
+		(layer "B.Cu")
+		(net "/I2C_SDA")
+	)
+	(segment
 		(start 85.960916 66.465625)
 		(end 85.722291 66.227)
@@
 	(segment
 		(start 52.675 77)
-		(end 49.5 77)
+		(end 52.08 77)
 		(width 0.2)
 		(layer "B.Cu")
@@
 	)
 	(via
-		(at 49.5 78)
-		(size 0.6)
-		(drill 0.3)
-		(layers "F.Cu" "B.Cu")
-		(net "/I2C_SCL")
-	)
-	(via
 		(at 75.067 67.972998)
 		(size 0.6)
@@
 	)
 	(segment
-		(start 50.5 79)
-		(end 49.5 78)
-		(width 0.2)
-		(layer "B.Cu")
-		(net "/I2C_SCL")
-	)
-	(segment
 		(start 90.993873 67.027)
 		(end 90.417276 67.603597)
@@
 	)
 	(segment
+		(start 52.62 79)
+		(end 47.5 84.12)
+		(width 0.2)
+		(layer "B.Cu")
+		(net "/I2C_SCL")
+	)
+	(segment
 		(start 88.918082 67.167015)
 		(end 88.609373 66.858306)
@@
 	(segment
 		(start 52.675 79)
-		(end 50.5 79)
-		(width 0.2)
-		(layer "B.Cu")
+		(end 52.62 79)
+		(width 0.2)
+		(layer "B.Cu")
